File: hardware/schematic/schematic.kicad_sch (KiCad schematic)
At the start: 3 parts, among them SW1 SW_SPST, U1 ESP32-C3-DevKitM-1

Commit message: Added button and led
Parts:
- added D1: LED, symbol Device:LED
- added R1: 1k, symbol Device:R_Small
- added SW2: SW_Push, symbol Switch:SW_Push
Connections:
- net GND: now also R1.1, SW2.2
- net ~{GPIO20-RESET}: now reaches U2.1 (~{RESET})
- net ~{GPIO20-RESET}: now also U1.28 (GPIO20/U0RXD)
- net at U1.10 (GPIO1): now also SW2.1
- net at U1.4 (GPIO2): now also D1.2 (A)
- net GP109-MP3CS renamed GP109-XCS
- new net: D1.1 (K), R1.2

Commit message: Changed power wiring
Connections:
- net 3V3: now also U2.2 (3V3)
Changed lines of the file:
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@@
+		)
+	)
+	(polyline
+		(pts
+			(xy 167.64 49.53) (xy 176.53 49.53)
+		)
+		(stroke
+			(width 0)
+			(type dash)
 		)
 	)
@@
 	(wire
 		(pts
+			(xy 82.55 30.48) (xy 181.61 30.48)
+		)
+		(stroke
+			(width 0)
+			(type default)
+		)
+	)
+	(wire
+		(pts
+			(xy 82.55 60.96) (xy 82.55 30.48)
+		)
+		(stroke
+			(width 0)
+			(type default)
+		)
+	)
+	(wire
+		(pts
 			(xy 113.03 99.06) (xy 133.35 99.06)
 		)
@@
 	(wire
 		(pts
+			(xy 181.61 30.48) (xy 181.61 58.42)
+		)
+		(stroke
+			(width 0)
+			(type default)
+		)
+	)
+	(wire
+		(pts
 			(xy 143.51 71.12) (xy 166.37 71.12)
 		)
@@
 		)
 	)
+	(polyline
+		(pts
+			(xy 182.88 33.02) (xy 191.77 33.02)
+		)
+		(stroke
+			(width 0)
+			(type dash)
+		)
+	)
 	(wire
 		(pts
@@
 	)
 	(rectangle
-		(start 53.34 48.26)
-		(end 100.33 58.42)
+		(start 83.82 48.26)
+		(end 130.81 58.42)
 		(stroke
 			(width 0)
@@
 		)
 	)
+	(text_box "Used to power \nthe amplifier\nalone\n"
+		(exclude_from_sim no)
+		(at 151.13 46.99 0)
+		(size 16.51 7.62)
+		(stroke
+			(width 0)
+			(type dash)
+		)
+		(fill
+			(type none)
+		)
+		(effects
+			(font
+				(size 1.27 1.27)
+			)
+			(justify left top)
+		)
+	)
+	(text_box "This assumes that the ESP32-C3-Devkit-M3 \nsupplies enough current for the VS1053"
+		(exclude_from_sim no)
+		(at 191.77 25.4 0)
+		(size 33.02 12.7)
+		(stroke
+			(width 0)
+			(type dash)
+		)
+		(fill
+			(type none)
+		)
+		(effects
+			(font
+				(size 1.27 1.27)
+			)
+			(justify left top)
+		)
+	)
 	(text "Open when USB connected!"
 		(exclude_from_sim no)
-		(at 70.104 53.848 0)
+		(at 114.554 53.848 0)
 		(effects
 			(font
