File: hardware/rotary-encoder/rotary-encoder.kicad_sch (KiCad schematic)
At the start: 15 parts, among them J1 Conn_01x05, J2 Conn_01x03

Commit message: Protoboard layout
Other:
- title: (none) -> "Analogue" Rotary Encoder circuit
Changed lines of the file:
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@@
 	(generator_version "9.0")
 	(paper "A4")
+	(title_block
+		(title "\"Analogue\" Rotary Encoder circuit")
+		(comment 1 "Only one MCU pin is used")
+	)
 	(text_box "External Board"
 		(exclude_from_sim no)
